File: ArcPad/macropad.kicad_sch (KiCad schematic)
At the start: 14 parts, among them J1 Conn_01x08_Pin, J2 Conn_01x04_Pin, SW1 SW_Push, SW10 SW_Push, SW11 SW_Push, SW2 SW_Push, SW3 SW_Push, SW4 SW_Push, SW5 SW_Push, SW6 SW_Push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

Commit message: small schematic change
Other:
- note added: "Raspberry Pi Pico 2 W"
- note removed: "Raspberry Pi Pico"
Changed lines of the file:
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@@
 		(company "Korv")
 	)
-	(text "Raspberry Pi Pico "
+	(text "Raspberry Pi Pico 2 W"
 		(exclude_from_sim no)
 		(at 38.608 20.574 0)
